File: VMU.brd (EAGLE design)
At the start: 16 parts

Commit message: general outline
Parts:
- moved SG1 36.8 mm to (66.6, 38.2)
- moved SG2 35.7 mm to (49.2, 38.2)
- moved BAT- 26.4 mm to (38.4, 52.5)
- moved BAT+ 20.8 mm to (38.3, 45.2)
- moved R1 17.7 mm to (38.0, 37.7), turned to 90 degrees
- moved S1 6.23 mm to (20.2, 58.6)
- moved RIGHT 5.69 mm to (14.0, 12.5)
- moved X 5.13 mm to (25.0, 9.00)
- moved UP 4.98 mm to (9.50, 16.0)
- moved DOWN 4.86 mm to (9.50, 7.50)
- moved MODE 3.57 mm to (29.0, 16.0)
- moved SLEEP 3.22 mm to (22.5, 16.0)
- moved LEFT 3.02 mm to (5.00, 12.5)
- moved Z 2.24 mm to (35.0, 10.0)
- moved PI1 2.04 mm to (35.0, 65.2)
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Other:
- board outline added: 40 x 60 mm
